Commit message: remove loadhand arguments, they are depracated

File: franka_description/robots/panda.transmission.xacro (robot description, xacro)
@@ -1,5 +1,5 @@
 <?xml version="1.0"?>
 <robot xmlns:xacro="http://www.ros.org/wiki/xacro">
-    <xacro:macro name="panda_transmission" params="robot_name load_hand">
+    <xacro:macro name="panda_transmission" params="robot_name">
         <!-- Load Gazebo lib and set the robot namespace -->
         <gazebo>
@@ -78,26 +78,24 @@
             </actuator>
         </transmission>
-        <xacro:if value="${load_hand}">
-            <transmission name="${robot_name}_leftfinger">
-                <type>transmission_interface/SimpleTransmission</type>
-                <joint name="${robot_name}_finger_joint1">
-                    <hardwareInterface>hardware_interface/VelocityJointInterface</hardwareInterface>
-                </joint>
-                <actuator name="${robot_name}_finger_joint1">
-                    <hardwareInterface>hardware_interface/VelocityJointInterface</hardwareInterface>
-                    <mechanicalReduction>1</mechanicalReduction>
-                </actuator>
-            </transmission>
-            <transmission name="${robot_name}_rightfinger">
-                <type>transmission_interface/SimpleTransmission</type>
-                <joint name="${robot_name}_finger_joint2">
-                    <hardwareInterface>hardware_interface/VelocityJointInterface</hardwareInterface>
-                </joint>
-                <actuator name="${robot_name}_finger_joint2">
-                    <hardwareInterface>hardware_interface/VelocityJointInterface</hardwareInterface>
-                    <mechanicalReduction>1</mechanicalReduction>
-                </actuator>
-            </transmission>
-        </xacro:if>
+        <transmission name="${robot_name}_leftfinger">
+            <type>transmission_interface/SimpleTransmission</type>
+            <joint name="${robot_name}_finger_joint1">
+                <hardwareInterface>hardware_interface/VelocityJointInterface</hardwareInterface>
+            </joint>
+            <actuator name="${robot_name}_finger_joint1">
+                <hardwareInterface>hardware_interface/VelocityJointInterface</hardwareInterface>
+                <mechanicalReduction>1</mechanicalReduction>
+            </actuator>
+        </transmission>
+        <transmission name="${robot_name}_rightfinger">
+            <type>transmission_interface/SimpleTransmission</type>
+            <joint name="${robot_name}_finger_joint2">
+                <hardwareInterface>hardware_interface/VelocityJointInterface</hardwareInterface>
+            </joint>
+            <actuator name="${robot_name}_finger_joint2">
+                <hardwareInterface>hardware_interface/VelocityJointInterface</hardwareInterface>
+                <mechanicalReduction>1</mechanicalReduction>
+            </actuator>
+        </transmission>
     </xacro:macro>
 </robot>

File: franka_description/robots/panda_arm.urdf.xacro (robot description, xacro)
@@ -10,5 +10,5 @@
   <xacro:arg name="robot_name" default="panda"/>
   <xacro:panda_gazebo robot_name="$(arg robot_name)" />
-  <xacro:panda_transmission robot_name="$(arg robot_name)" load_hand="false" />
+  <xacro:panda_transmission robot_name="$(arg robot_name)"/>
   <!-- end for simulation -->
 </robot>

File: franka_description/robots/panda_arm_hand.urdf.xacro (robot description, xacro)
@@ -12,5 +12,5 @@
   <xacro:arg name="robot_name" default="panda"/>
   <xacro:panda_gazebo robot_name="$(arg robot_name)" />
-  <xacro:panda_transmission robot_name="$(arg robot_name)" load_hand="true" />
+  <xacro:panda_transmission robot_name="$(arg robot_name)" />
   <!-- end for simulation -->
 </robot>
